Commit message: add_slope_input

File: urdf/L580_end_link.xacro (robot description, xacro)
@@ -13,14 +13,21 @@
     <inertial>
       <mass value="5000.0"/>
-      <origin xyz="-2.61002 0.0 -0.48814" rpy="0 0 0"/>
+      <origin xyz="-2.35168  0.0 -0.48814" rpy="0 0 0"/>
       <inertia ixx="5000.0" ixy="0.0" ixz="500.0" iyy="15000.0" iyz="0.0" izz="13000.0"/>
     </inertial>
-    <visual><geometry><mesh filename="file:///$(find loader_sim_pkg)/meshes/body.STL"/></geometry><material name="yellow"/></visual>
-    <collision><geometry><mesh filename="file:///$(find loader_sim_pkg)/meshes/body.STL"/></geometry></collision>
+    <visual>
+      <origin xyz="0.25834 0 0" rpy="0 0 0"/>
+      <geometry><mesh filename="file:///$(find loader_sim_pkg)/meshes/body.STL"/></geometry>
+      <material name="yellow"/>
+    </visual>
+    <collision>
+      <origin xyz="0.25834 0 0" rpy="0 0 0"/>
+      <geometry><mesh filename="file:///$(find loader_sim_pkg)/meshes/body.STL"/></geometry>
+    </collision>
   </link>
   <joint name="front_wheel_joint" type="continuous">
     <parent link="base_link"/>
     <child link="front_wheel_link"/>
-    <origin xyz="0.43775 0 -1.5816" rpy="-1.57 -1.57 0"/>
+    <origin xyz="0.69609 0 -1.5816" rpy="-1.57 -1.57 0"/>
     <axis xyz="0 0 1"/>
   </joint>
@@ -37,5 +44,5 @@
     <parent link="base_link"/>
     <child link="rear_wheel_link"/>
-    <origin xyz="-3.33631 0 -1.5816" rpy="-1.57 -1.57 0"/>
+    <origin xyz="-3.07797 0 -1.5816" rpy="-1.57 -1.57 0"/>
     <axis xyz="0 0 1"/>
   </joint>
@@ -52,5 +59,5 @@
     <parent link="base_link"/>
     <child link="arm_link1"/>
-    <origin xyz="-0.25834 0 0.08169" rpy="-1.57 0 0"/> <!-- rpy="-1.57 0.40815617 0" -->
+    <origin xyz="0 0 0.08169" rpy="-1.57 0 0"/> <!-- rpy="-1.57 0.40815617 0" -->
     <axis xyz="0 0 1"/>
     <limit lower="-1.5" upper="1.5" effort="50000" velocity="0.5"/>
@@ -137,6 +144,6 @@
             <slip1>0.0</slip1>
             <slip2>0.0</slip2>
-            <mu>1.2</mu>
-            <mu2>1.2</mu2>
+            <mu>10.0</mu>
+            <mu2>10.0</mu2>
           </ode>
         </friction>
@@ -150,6 +157,6 @@
             <slip1>0.0</slip1>
             <slip2>0.0</slip2>
-            <mu>1.2</mu>
-            <mu2>1.2</mu2>
+            <mu>10.0</mu>
+            <mu2>10.0</mu2>
           </ode>
         </friction>
